File: pcb/hackpad.kicad_pcb (KiCad board)
At the start: 2 copper layers, 76.2 x 83.8 mm, 33 parts, among them SW1 SW_Push, SW10 RotaryEncoder_Switch, SW2 SW_Push, SW4 SW_Push, SW5 SW_Push, SW6 SW_Push, SW7 SW_Push, SW8 SW_Push, SW9 SW_Push, U1 MOUDLE-SEEEDUINO-XIAO, U2 ER_OLEDM0.91_1x-I2C

Commit message: adding case and updating the pcb
make hole for scren in pcb and adding silk screen image in pcb.
Parts:
- removed C1: C_Small, Capacitor_THT:CP_Radial_D5.0mm_P2.00mm
- added G***: LOGO, hacklcublogofootprint:hackclub flag, B.Cu at (117.8, 128.1)
- added G***: OrpheusHackClubIcon, SKS:OrpheusHackClubIcon, B.Cu at (157.6, 70.7)
- moved D3 7.92 mm to (155.6, 83.5), turned to -90 degrees
- moved SW10 0.94 mm to (173.6, 88.0)
- moved D21 0.94 mm to (165.1, 95.5)
Routing:
- net VDD: track 315.1 -> 302.1 mm
- net Net-(D3-A): track 4.17 -> 9.84 mm
- net GND: track 390.0 -> 385.1 mm
- net Row1: track 71.4 -> 73.6 mm
- net Rotary A: track 84.3 -> 85.4 mm
- net Rotary B: track 76.1 -> 77.0 mm
- net Column1: track 73.5 -> 72.8 mm
Other:
- outline, holes or cut-outs redrawn
- board text added: "RX-pad"
- board text added: "Sandwich"
