File: pcb/hackpad.kicad_sch (KiCad schematic)
At the start: 0 parts

Commit message: Create the pcb
Adding 3d part to the footprint
and fixing the schematic
Parts:
- added C1: C_Small, Capacitor_THT:CP_Radial_D5.0mm_P2.00mm, symbol Device:C_Small
- added D1, D2, D3, D4, D5, D6, D7, D8, D9: 1N4148, Diode_THT:D_DO-35_SOD27_P7.62mm_Horizontal, symbol Diode:1N4148
- added D10, D11, D12, D13, D14, D15, D16, D17, D18, D19, D20, D21: SK6812MINI-E, LED_SMD:LED_SK6812MINI-E_3.2x2.8mm_P1.5mm_ReverseMount, symbol LED:SK6812MINI-E
- added SW1, SW2, SW4, SW5, SW6, SW7, SW8, SW9: SW_Push, Button_Switch_Keyboard:SW_Cherry_MX_1.00u_PCB, symbol Switch:SW_Push
- added SW10: RotaryEncoder_Switch, Rotary_Encoder:RotaryEncoder_Alps_EC11E-Switch_Vertical_H20mm, symbol Device:RotaryEncoder_Switch
- added U1: MOUDLE-SEEEDUINO-XIAO, footprints:XIAO-Generic-Hybrid-14P-2.54-21X17.8MM, symbol XIAO_RP2040:MOUDLE-SEEEDUINO-XIAO
- added U2: ER_OLEDM0.91_1x-I2C, Display:ER_OLEDM0.91_1x-I2C, symbol Display_Graphic:ER_OLEDM0.91_1x-I2C
Connections:
- new net: D14.4 (DOUT), D15.2 (DIN)
- new net: D15.4 (DOUT), D16.2 (DIN)
- new net: D1.2 (A), SW1.2
- new net: D18.4 (DOUT), D19.2 (DIN)
- new net: D19.4 (DOUT), D20.2 (DIN)
- new net: D13.4 (DOUT), D14.2 (DIN)
- new net: D5.2 (A), SW5.2
- new net: D8.2 (A), SW8.2
- new net: D7.2 (A), SW7.2
- new net: D3.2 (A), SW10.S1
- new net: D4.2 (A), SW4.2
- new net: D12.4 (DOUT), D13.2 (DIN)
- new net: D20.4 (DOUT), D21.2 (DIN)
- new net: D2.2 (A), SW2.2
- new net: D10.4 (DOUT), D11.2 (DIN)
- new net: D11.4 (DOUT), D12.2 (DIN)
- new net: D6.2 (A), SW6.2
- new net: D16.4 (DOUT), D17.2 (DIN)
- new net: D17.4 (DOUT), D18.2 (DIN)
- new net: D9.2 (A), SW9.2
- new net Column1: SW1.1, SW4.1, SW7.1, U1.3 (PA10_A2_D2)
- new net Column2: SW2.1, SW5.1, SW8.1, U1.4 (PA11_A3_D3)
- new net Column3: SW10.S2, SW6.1, SW9.1, U1.7 (PB08_A6_D6_TX)
- new net GND: C1.2, D10.1 (VSS), D11.1 (VSS), D12.1 (VSS), D13.1 (VSS), D14.1 (VSS), D15.1 (VSS), D16.1 (VSS), D17.1 (VSS), D18.1 (VSS), D19.1 (VSS), D20.1 (VSS), D21.1 (VSS), SW10.C, U1.13 (GND), U2.1 (GND)
- new net Led DIN: D10.2 (DIN), U1.11 (PA6_A10_D10_MOSI)
- new net Rotary A: SW10.A, U1.1 (PA02_A0_D0)
- new net Rotary B: SW10.B, U1.2 (PA4_A1_D1)
- new net Row1: D1.1 (K), D2.1 (K), D3.1 (K), U1.8 (PB09_A7_D7_RX)
- new net Row2: D4.1 (K), D5.1 (K), D6.1 (K), U1.9 (PA7_A8_D8_SCK)
- new net Row3: D7.1 (K), D8.1 (K), D9.1 (K), U1.10 (PA5_A9_D9_MISO)
- new net SCL: U1.6 (PA9_A5_D5_SCL), U2.3 (SCL)
- new net SDA: U1.5 (PA8_A4_D4_SDA), U2.4 (SDA)
- new net VCC: U1.12 (3V3), U2.2 (VCC)
- new net VDD: C1.1, D10.3 (VDD), D11.3 (VDD), D12.3 (VDD), D13.3 (VDD), D14.3 (VDD), D15.3 (VDD), D16.3 (VDD), D17.3 (VDD), D18.3 (VDD), D19.3 (VDD), D20.3 (VDD), D21.3 (VDD), U1.14 (5V)
- no-connect marks 0 -> 1
Other:
- note added: "RX-pad"

Commit message: adding case and updating the pcb
make hole for scren in pcb and adding silk screen image in pcb.
Parts:
- removed C1: C_Small, Capacitor_THT:CP_Radial_D5.0mm_P2.00mm, symbol Device:C_Small
Changed lines of the file:
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@@
-	)
-	(junction
-		(at 44.45 151.13)
-		(diameter 0)
-		(color 0 0 0 0)
 	)
 	(junction
@@
 		(color 0 0 0 0)
 	)
-	(junction
-		(at 44.45 123.19)
-		(diameter 0)
-		(color 0 0 0 0)
-	)
 	(no_connect
 		(at 269.24 137.16)
@@
 	(wire
 		(pts
-			(xy 44.45 134.62) (xy 44.45 151.13)
-		)
-		(stroke
-			(width 0)
-			(type default)
-		)
-	)
-	(wire
-		(pts
-			(xy 34.29 151.13) (xy 44.45 151.13)
+			(xy 34.29 151.13) (xy 54.61 151.13)
 		)
 		(stroke
@@
 	(wire
 		(pts
-			(xy 44.45 123.19) (xy 54.61 123.19)
+			(xy 36.83 123.19) (xy 54.61 123.19)
 		)
 		(stroke
@@
 	(wire
 		(pts
-			(xy 44.45 123.19) (xy 44.45 129.54)
-		)
-		(stroke
-			(width 0)
-			(type default)
-		)
-	)
-	(wire
-		(pts
 			(xy 160.02 58.42) (xy 160.02 69.85)
 		)
@@
 	(wire
 		(pts
-			(xy 36.83 123.19) (xy 44.45 123.19)
-		)
-		(stroke
-			(width 0)
-			(type default)
-		)
-	)
-	(wire
-		(pts
 			(xy 172.72 123.19) (xy 190.5 123.19)
 		)
@@
 		(pts
 			(xy 172.72 151.13) (xy 190.5 151.13)
-		)
-		(stroke
-			(width 0)
-			(type default)
-		)
-	)
-	(wire
-		(pts
-			(xy 44.45 151.13) (xy 54.61 151.13)
 		)
 		(stroke
@@
 					(unit 1)
 				)
-			)
-		)
-	)
-	(symbol
-		(lib_id "Device:C_Small")
-		(at 44.45 132.08 0)
-		(unit 1)
-		(body_style 1)
-		(exclude_from_sim no)
-		(in_bom yes)
-		(on_board yes)
-		(in_pos_files yes)
-		(dnp no)
-		(fields_autoplaced yes)
-		(property "Reference" "C1"
-			(at 46.99 130.8099 0)
-			(show_name no)
-			(do_not_autoplace no)
-			(effects
-				(font
-					(size 1.27 1.27)
-				)
-				(justify left)
-			)
-		)
-		(property "Value" "C_Small"
-			(at 46.99 133.3499 0)
-			(show_name no)
-			(do_not_autoplace no)
-			(effects
-				(font
-					(size 1.27 1.27)
-				)
-				(justify left)
-			)
-		)
-		(property "Footprint" "Capacitor_THT:CP_Radial_D5.0mm_P2.00mm"
-			(at 44.45 132.08 0)
-			(hide yes)
-			(show_name no)
-			(do_not_autoplace no)
-			(effects
-				(font
-					(size 1.27 1.27)
-				)
-			)
-		)
-		(property "Datasheet" ""
-			(at 44.45 132.08 0)
-			(hide yes)
-			(show_name no)
-			(do_not_autoplace no)
-			(effects
-				(font
-					(size 1.27 1.27)
-				)
-			)
-		)
-		(property "Description" "Unpolarized capacitor, small symbol"
-			(at 44.45 142.24 0)
-			(hide yes)
-			(show_name no)
-			(do_not_autoplace no)
-			(effects
-				(font
-					(size 1.27 1.27)
-				)
-			)
-		)
-		(pin "1"
-		)
-		(pin "2"
-		)
-		(instances
-			(project "hackpad"
-				(path "/22d8b9f8-be1c-41e1-8107-8ea76f2ee119"
-					(reference "C1")
-					(unit 1)
-				)
